File: opendeck-board/opendeck.kicad_sch (KiCad schematic)
At the start: 73 parts

Commit message: added the matrices, leds and crossfader
Parts:
- added D1, D10, D11, D12, D13, D14, D15, D16, D2, D3, D4, D5, D6, D7, D8, D9: WS2812B, LED_SMD:LED_WS2812B_PLCC4_5.0x5.0mm_P3.2mm, symbol LED:WS2812B
- added D49, D50, D51, D52, D53, D54, D55, D56, D57, D58, D59, D60, D61, D62, D63, D64, D65, D66: D, symbol Device:D
- added R1, R34, R35, R36: 1K, symbol Device:R
- added RV1: POT_vol_L, symbol Device:R_Potentiometer
- added RV10, RV11, RV8, RV9: R_Potentiometer, symbol Device:R_Potentiometer
- added RV2: POT_vol_R, symbol Device:R_Potentiometer
- added RV3: POT_crossfader, symbol Device:R_Potentiometer
- added SW1, SW10, SW11, SW12, SW13, SW14, SW15, SW16, SW17, SW18, SW2, SW3, SW4, SW5, SW6, SW7, SW8, SW9, filter_sw_L, filter_sw_L1, hearphone_sw_L, hearphone_sw_R: SW_SPST, symbol Switch:SW_SPST
- gave numbers to parts that had none: 73
Connections:
- net +3V3: now also RV10.1, RV11.1, RV8.1, RV9.1, filter_sw_L.2 (B), filter_sw_L1.2 (B)
- net GND: now also D1.1 (VDD), D10.1 (VDD), D11.1 (VDD), D12.1 (VDD), D13.1 (VDD), D14.1 (VDD), D15.1 (VDD), D16.1 (VDD), D2.1 (VDD), D3.1 (VDD), D4.1 (VDD), D5.1 (VDD), D6.1 (VDD), D7.1 (VDD), D8.1 (VDD), D9.1 (VDD), R1.2, R34.2, R35.2, R36.2, RV1.3, RV10.3, RV11.3, RV2.3, RV3.1, RV8.3, RV9.3
- new net: D64.1 (K), SW16.1 (A)
- new net: D15.4 (DIN), D16.2 (DOUT)
- new net: D52.1 (K), SW4.1 (A)
- new net: D65.1 (K), SW17.1 (A)
- new net: D53.1 (K), SW5.1 (A)
- new net: D61.1 (K), SW13.1 (A)
- new net: D60.1 (K), SW12.1 (A)
- new net: D11.4 (DIN), D12.2 (DOUT)
- new net: D12.4 (DIN), D13.2 (DOUT)
- new net: D57.1 (K), SW9.1 (A)
- new net: D3.2 (DOUT), D4.4 (DIN)
- new net: D2.2 (DOUT), D3.4 (DIN)
- new net: D54.1 (K), SW6.1 (A)
- new net: D55.1 (K), SW7.1 (A)
- new net: R34.1, hearphone_sw_R.1 (A)
- new net: D59.1 (K), SW11.1 (A)
- new net: D10.2 (DOUT), D9.4 (DIN)
- new net: D13.4 (DIN), D14.2 (DOUT)
- new net: R1.1, filter_sw_L.1 (A)
- new net: D5.4 (DIN), D6.2 (DOUT)
- new net: D51.1 (K), SW3.1 (A)
- new net: D6.4 (DIN), D7.2 (DOUT)
- new net: D1.2 (DOUT), D2.4 (DIN)
- new net: D14.4 (DIN), D15.2 (DOUT)
- new net: R36.1, filter_sw_L1.1 (A)
- new net: D56.1 (K), SW8.1 (A)
- new net: D4.2 (DOUT), D8.4 (DIN)
- new net: R35.1, hearphone_sw_L.1 (A)
- new net: D10.4 (DIN), D11.2 (DOUT)
- new net: D62.1 (K), SW14.1 (A)
- new net: D63.1 (K), SW15.1 (A)
- new net: D7.4 (DIN), D8.2 (DOUT)
- new net: D66.1 (K), SW18.1 (A)
- new net: D58.1 (K), SW10.1 (A)
- new net: D50.1 (K), SW2.1 (A)
- new net: D49.1 (K), SW1.1 (A)
- new net +3.3V: RV1.1, RV2.1, RV3.3, hearphone_sw_L.2 (B), hearphone_sw_R.2 (B)
- new net +5V: D1.3 (VSS), D10.3 (VSS), D11.3 (VSS), D12.3 (VSS), D13.3 (VSS), D14.3 (VSS), D15.3 (VSS), D16.3 (VSS), D2.3 (VSS), D3.3 (VSS), D4.3 (VSS), D5.3 (VSS), D6.3 (VSS), D7.3 (VSS), D8.3 (VSS), D9.3 (VSS)
- new net dpad_column_A: SW1.2 (B), SW4.2 (B), SW7.2 (B)
- new net dpad_column_B: SW2.2 (B), SW5.2 (B), SW8.2 (B)
- new net dpad_column_C: SW3.2 (B), SW6.2 (B), SW9.2 (B)
- new net dpad_column_D: SW10.2 (B), SW11.2 (B), SW12.2 (B)
- new net dpad_column_E: SW13.2 (B), SW14.2 (B), SW15.2 (B)
- new net dpad_column_F: SW16.2 (B), SW17.2 (B), SW18.2 (B)
- new net dpad_row_1: D49.2 (A), D50.2 (A), D51.2 (A), D58.2 (A), D61.2 (A), D64.2 (A)
- new net dpad_row_2: D52.2 (A), D53.2 (A), D54.2 (A), D59.2 (A), D62.2 (A), D65.2 (A)
- new net dpad_row_3: D55.2 (A), D56.2 (A), D57.2 (A), D60.2 (A), D63.2 (A), D66.2 (A)
- new net padsLED_L: D1.4 (DIN)
- new net padsLED_R: D16.4 (DIN)
Other:
- moved on the sheet: RV4, RV5, RV6, RV7

Commit message: Adding more rows to the button matrix and moving the center module buttons to it
Parts:
- removed R1, R34, R35, R36: 1K, symbol Device:R
- removed filter_sw_L1: SW_SPST, symbol Switch:SW_SPST
- added D68, D69, D71, D72, D73, D74, D75, D76, D79: D, symbol Device:D
- added SW20, SW21, SW23, SW24, filter_sw_R, shift_switch: SW_SPST, symbol Switch:SW_SPST
Connections:
- net +3.3V: no longer hearphone_sw_L.2 (B), hearphone_sw_R.2 (B)
- net +3V3: no longer filter_sw_L.2 (B)
- net dpad_column_A: now also hearphone_sw_L.2 (B), SW23.2 (B), SW24.2 (B); no longer SW1.2 (B), SW4.2 (B), SW7.2 (B)
- net dpad_column_B: now also SW7.2 (B), SW9.2 (B); no longer SW2.2 (B), SW5.2 (B)
- net dpad_column_C: now also SW4.2 (B), SW5.2 (B); no longer SW3.2 (B), SW9.2 (B)
- net dpad_column_D: now also SW1.2 (B), SW2.2 (B), SW3.2 (B); no longer SW10.2 (B), SW11.2 (B), SW12.2 (B)
- net dpad_column_E: now also SW16.2 (B), SW17.2 (B), SW18.2 (B); no longer SW13.2 (B), SW14.2 (B), SW15.2 (B)
- net dpad_column_F: now also SW13.2 (B), SW14.2 (B), SW15.2 (B); no longer SW16.2 (B), SW17.2 (B), SW18.2 (B)
- net dpad_row_1: now also D52.2 (A), D55.2 (A), D73.2 (A), D76.2 (A), D79.2 (A); no longer D50.2 (A), D51.2 (A)
- net dpad_row_2: now also D50.2 (A), D56.2 (A), D68.2 (A), D71.2 (A), D74.2 (A); no longer D52.2 (A), D54.2 (A)
- net dpad_row_3: now also D51.2 (A), D54.2 (A), D69.2 (A), D72.2 (A), D75.2 (A); no longer D55.2 (A), D56.2 (A)
- net at hearphone_sw_R.1 (A): now also D79.1 (K)
- net at filter_sw_L.1 (A): now also D73.1 (K)
- net at hearphone_sw_L.1 (A): now also D76.1 (K)
- new net: D71.1 (K), SW23.1 (A)
- new net: D69.1 (K), SW21.1 (A)
- new net: D74.1 (K), filter_sw_R.1 (A)
- new net: D68.1 (K), SW20.1 (A)
- new net: D72.1 (K), SW24.1 (A)
- new net: D75.1 (K), shift_switch.1 (A)
- new net dpad_column_G: SW10.2 (B), SW11.2 (B), SW12.2 (B)
- new net dpad_column_H: SW20.2 (B), SW21.2 (B), hearphone_sw_R.2 (B)
- new net dpad_column_I: filter_sw_L.2 (B), filter_sw_R.2 (B), shift_switch.2 (B)
Other:
- moved on the sheet: D1, D10, D11, D12, D13, D14, D15, D16, D17, D18, D19, D2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

Commit message: Added the pots and keypad to the teensy
Parts:
- added D67, D70, D77, D78, D80, D81: D, symbol Device:D
- added SW19, SW22, SW25, SW26, SW27, SW28: SW_SPST, symbol Switch:SW_SPST
Connections:
- net dpad_column_A: now also U3.7 (5_TX1_MISO1)
- net dpad_column_B: now also U3.8 (6_RX3_CS1_PWM), SW26.2 (B), SW27.2 (B), SW28.2 (B)
- net dpad_column_C: now also U3.9 (7_RX3_MOSI0)
- net dpad_column_D: now also U3.10 (8_TX3_MISO0)
- net dpad_column_E: now also U3.11 (9_RX2_PWM)
- net dpad_column_F: now also U3.12 (10_TX2_CS0_PWM)
- net dpad_column_G: now also U3.13 (11_MOSI0), SW19.2 (B), SW22.2 (B), SW25.2 (B)
- net dpad_column_H: now also U3.14 (12_MISO0)
- net dpad_column_I: now also U3.20 (13_LED_SCK0)
- net dpad_row_1: now also U3.3 (1_TX1_MISO1_Touch), D67.2 (A), D78.2 (A)
- net dpad_row_2: now also U3.5 (3_RX1_PWM_Touch), D70.2 (A), D80.2 (A)
- net dpad_row_3: now also U3.6 (4_TX1_PWM_Touch), D77.2 (A), D81.2 (A)
- net A10: now reaches RV11.2
- net A10: now also U3.19 (26_A12/DAC)
- net A7: now reaches RV8.2
- net A7: now also U3.28 (21_A7_MOSI1_RX1)
- net A8: now reaches RV9.2
- net A8: now also U3.29 (22_A8_SCL1_PWM_Touch)
- net A9: now reaches RV10.2
- net A9: now also U3.30 (23_A9_SDA1_PWM_Touch)
- net A6: now reaches RV7.2
- net A6: now also U3.27 (20_A6_SCK1_PWM_TX3)
- net A3: now reaches RV4.2
- net A3: now also U3.24 (17_A3_SDA0_PWM_Touch)
- net A1: now reaches RV1.2
- net A1: now also U3.22 (15_A1_Touch)
- net A4: now reaches RV5.2
- net A4: now also U3.25 (18_A4_SDA0_Touch)
- net A2: now reaches RV2.2
- net A2: now also U3.23 (16_A2_SCL0_PWM_Touch)
- net A0: now reaches U3.21 (14_A0_SCK0)
- net A0: now also RV3.2
- net A5: now reaches U3.26 (19_A5_SCL0_Touch)
- net A5: now also RV6.2
- new net: D78.1 (K), SW26.1 (A)
- new net: D77.1 (K), SW25.1 (A)
- new net: D81.1 (K), SW28.1 (A)
- new net: D80.1 (K), SW27.1 (A)
- new net: D70.1 (K), SW22.1 (A)
- new net: D67.1 (K), SW19.1 (A)
Other:
- moved on the sheet: RV1, RV10, RV11, RV2, RV3, RV4, RV5, RV6, RV7, RV8, RV9
