File: opendeck-board/opendeck_sides/side_board/side_board.kicad_pcb (KiCad board)
At the start: 2 copper layers, 30 parts, among them SW1 SW_SPST, SW10 SW_SPST, SW11 SW_SPST, SW2 SW_SPST, SW3 SW_SPST, SW4 SW_SPST, SW5 SW_SPST, SW6 SW_SPST, SW7 SW_SPST, SW8 SW_SPST, SW9 SW_SPST

Commit message: creating the side board
Parts:
- added D20: WS2812B, LED_SMD:LED_WS2812B_PLCC4_5.0x5.0mm_P3.2mm, F.Cu at (104.1, 128.3)
- added D21: WS2812B, LED_SMD:LED_WS2812B_PLCC4_5.0x5.0mm_P3.2mm, F.Cu at (132.1, 128.3)
- added D22: WS2812B, LED_SMD:LED_WS2812B_PLCC4_5.0x5.0mm_P3.2mm, F.Cu at (160.1, 128.3)
- added J1: Conn_01x10_Male, Connector_IDC:IDC-Header_2x05_P2.54mm_Horizontal, F.Cu at (58.4, 54.0)
- D10, D11, D12, D13, D14, D15, D16, D17, D18, D19, D9: footprint Diode_THT:D_5KPW_P12.70mm_Horizontal -> Diode_THT:D_5W_P12.70mm_Horizontal
- SW1, SW10, SW11, SW2, SW3, SW4, SW5, SW6, SW7, SW8, SW9: footprint Button_Switch_Keyboard:SW_Cherry_MX_1.00u_PCB -> Library:SW_Cherry_MX_1.00u_PCB_3d
- moved SW8 172.8 mm to (78.7, 109.2)
- moved SW4 160.9 mm to (78.7, 81.3)
- moved SW10 134.9 mm to (134.6, 109.2)
- moved SW6 115.7 mm to (134.6, 81.3)
- moved SW11 107.0 mm to (162.6, 109.2)
- moved SW9 106.8 mm to (106.7, 109.2)
- moved D8 106.7 mm to (76.2, 128.3), turned to 90 degrees
- moved SW7 94.3 mm to (162.6, 81.3)
- moved D4 84.1 mm to (76.2, 100.3), turned to 90 degrees
- moved D12 69.7 mm to (88.9, 81.3), turned to -90 degrees
- moved D16 67.7 mm to (88.9, 109.2), turned to -90 degrees
- moved D9 61.1 mm to (106.7, 50.8), turned to -90 degrees
- moved D5 55.4 mm to (104.2, 100.3), turned to 90 degrees
- moved D6 55.3 mm to (132.1, 100.3), turned to 90 degrees
- moved D10 48.3 mm to (132.1, 50.8), turned to -90 degrees
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Connections:
- D8 pad 2: unconnected-(D8-DOUT-Pad2) -> Net-(D20-DIN)
Routing:
- net +5V: track 0.00 -> 406.5 mm
- net GND: track 0.00 -> 388.7 mm
- net dpad_row_2: track 0.00 -> 362.3 mm, vias 0 -> 6
- net dpad_row_3: track 0.00 -> 308.3 mm
- net dpad_row_1: track 0.00 -> 262.7 mm, vias 0 -> 4
- net dpad_column_G: track 0.00 -> 174.0 mm
- net dpad_column_H: track 0.00 -> 160.9 mm
- net Net-(D7-DOUT): track 0.00 -> 123.9 mm
- net Net-(D3-DOUT): track 0.00 -> 112.0 mm
- net dpad_column_F: track 0.00 -> 88.4 mm
- net dpad_column_E: track 0.00 -> 72.6 mm
- net padsLED_R: track 0.00 -> 37.2 mm
- net Net-(D21-DOUT): track 0.00 -> 26.9 mm
- net Net-(D20-DOUT): track 0.00 -> 26.8 mm
- net Net-(D4-DOUT): track 0.00 -> 26.8 mm
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