File: opendeck-board/opendeck_sides/side_board/side_board.kicad_sch (KiCad schematic)
At the start: 30 parts, among them SW1 SW_SPST, SW10 SW_SPST, SW11 SW_SPST, SW2 SW_SPST, SW3 SW_SPST, SW4 SW_SPST, SW5 SW_SPST, SW6 SW_SPST, SW7 SW_SPST, SW8 SW_SPST, SW9 SW_SPST

Commit message: creating the side board
Parts:
- added D20, D21, D22: WS2812B, LED_SMD:LED_WS2812B_PLCC4_5.0x5.0mm_P3.2mm, symbol LED:WS2812B
- added J1: Conn_01x10_Male, Connector_IDC:IDC-Header_2x05_P2.54mm_Horizontal, symbol Connector:Conn_01x10_Male
- D10, D11, D12, D13, D14, D15, D16, D17, D18, D19, D9: footprint Diode_THT:D_5KPW_P12.70mm_Horizontal -> Diode_THT:D_5W_P12.70mm_Horizontal
- SW1, SW10, SW11, SW2, SW3, SW4, SW5, SW6, SW7, SW8, SW9: footprint Button_Switch_Keyboard:SW_Cherry_MX_1.00u_PCB -> Library:SW_Cherry_MX_1.00u_PCB_3d
Connections:
- net +5V: now also D20.3 (VSS), D21.3 (VSS), D22.3 (VSS), J1.2 (Pin_2)
- net GND: now also D20.1 (VDD), D21.1 (VDD), D22.1 (VDD), J1.1 (Pin_1)
- net dpad_column_E: now also J1.9 (Pin_9)
- net dpad_column_F: now also J1.7 (Pin_7)
- net dpad_column_G: now also J1.5 (Pin_5)
- net dpad_column_H: now also J1.3 (Pin_3)
- net dpad_row_1: now also J1.8 (Pin_8)
- net dpad_row_2: now also J1.6 (Pin_6)
- net dpad_row_3: now also J1.4 (Pin_4)
- net padsLED_R: now also J1.10 (Pin_10)
- net at D8.2 (DOUT): now also D20.4 (DIN)
- new net: D21.2 (DOUT), D22.4 (DIN)
- new net: D20.2 (DOUT), D21.4 (DIN)
Other:
- moved on the sheet: D1, D2, D3, D4, D5, D6, D7, D8
