File: opendeck-board/opendeck_center/opendeck_center.kicad_sch (KiCad schematic)
At the start: 162 parts, among them SW1 SW_SPST, SW10 SW_SPST, SW11 SW_SPST, SW12 SW_SPST, SW13 SW_SPST, SW14 SW_SPST, SW15 SW_SPST, SW16 SW_SPST, SW17 SW_SPST, SW18 SW_SPST, SW19 SW_SPST, SW2 SW_SPST, SW20 SW_SPST, SW21 SW_SPST, SW22 SW_SPST, SW23 SW_SPST, SW24 SW_SPST, SW25 SW_SPST, SW26 SW_SPST, SW27 SW_SPST, SW28 SW_SPST, SW3 SW_SPST, SW4 SW_SPST, SW5 SW_SPST, SW6 SW_SPST, SW7 SW_SPST, SW8 SW_SPST, SW9 SW_SPST, U1 74HC595, U2 74HC595, U3 Teensy-LC, U4 74HC595, U5 74HC595

Commit message: updating the I2C connections on the teensy
Parts:
- added C1, C2: 22pF, symbol Device:C
- added U6: ATmega328-P, Package_DIP:DIP-28_W7.62mm, symbol MCU_Microchip_ATmega:ATmega328-P
- added Y1: Crystal, symbol Device:Crystal
Connections:
- net A4: now also U3.36 (24_A10); no longer U3.25 (18_A4_SDA0_Touch)
- net A5: now also U3.37 (25_A11); no longer U3.26 (19_A5_SCL0_Touch)
- net GND: now also C1.2, C2.2
- new net: C1.1, U6.10 (XTAL2/PB7), Y1.1
- new net: C2.1, U6.9 (XTAL1/PB6), Y1.2
- new net: U6.22 (GND), U6.8 (GND)
- new net SCL: U3.26 (19_A5_SCL0_Touch), U6.28 (PC5)
- new net SDA: U3.25 (18_A4_SDA0_Touch), U6.27 (PC4)
